File: BarometerBoard.kicad_pcb (KiCad board)
At the start: 4 copper layers, 13.2 x 19.5 mm, 12 parts, among them J1 Conn_01x04_Pin, U6 MS5611-01BA

Commit message: Commit
Parts:
- added G***: LOGO, iclr:iclr_logo_estd2018_10mm, B.Cu at (123.5, 80.8)
- added J2: Conn_01x04_Pin, Connector_JST:JST_SH_SM04B-SRSS-TB_1x04-1MP_P1.00mm_Horizontal, F.Cu at (125.3, 80.9)
- moved G*** 9.24 mm to (124.7, 88.0), turned to 90 degrees
Routing:
- net /SCLK: track 12.2 -> 14.7 mm
- net /SDA: track 13.7 -> 16.2 mm
- net +3V3: track 2.63 -> 3.93 mm, vias 4 -> 5
- net GND: vias 8 -> 20
Other:
- board size 13.2 x 19.5 mm -> 19.9 x 19.5 mm
- board text added: "v1.0"
