File: BarometerBoard.kicad_sch (KiCad schematic)
At the start: 11 parts, among them J1 Conn_01x04_Pin, U6 MS5611-01BA

Commit message: Commit
Parts:
- added J2: Conn_01x04_Pin, Connector_JST:JST_SH_SM04B-SRSS-TB_1x04-1MP_P1.00mm_Horizontal, symbol Connector:Conn_01x04_Pin
Connections:
- net +3V3: now also J2.2 (Pin_2)
- net GND: now also J2.1 (Pin_1)
- net SCLK: now also J2.4 (Pin_4)
- net SDA: now also J2.3 (Pin_3)
Changed lines of the file:
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@@
+    (stroke (width 0) (type default))
+  )
+  (wire (pts (xy 156.718 61.976) (xy 153.67 61.976))
     (stroke (width 0) (type default))
   )
@@
   )
   (wire (pts (xy 226.568 51.562) (xy 226.568 54.102))
+    (stroke (width 0) (type default))
+  )
+  (wire (pts (xy 153.67 64.516) (xy 156.464 64.516))
     (stroke (width 0) (type default))
   )
@@
     (effects (font (size 1.27 1.27)) (justify left bottom))
   )
+  (label "SDA" (at 153.67 67.056 0) (fields_autoplaced)
+    (effects (font (size 1.27 1.27)) (justify left bottom))
+  )
   (label "SCLK" (at 191.262 107.188 0) (fields_autoplaced)
     (effects (font (size 1.27 1.27)) (justify left bottom))
@@
     (effects (font (size 1.27 1.27)) (justify right bottom))
   )
+  (label "SCLK" (at 153.67 69.596 0) (fields_autoplaced)
+    (effects (font (size 1.27 1.27)) (justify left bottom))
+  )
   (label "SDA" (at 191.262 101.854 0) (fields_autoplaced)
     (effects (font (size 1.27 1.27)) (justify left bottom))
@@
     )
   )
+  (symbol (lib_id "power:+3.3V") (at 156.464 64.516 0) (unit 1)
+    (in_bom yes) (on_board yes) (dnp no)
+    (property "Reference" "#PWR08" (at 156.464 68.326 0)
+      (effects (font (size 1.27 1.27)) hide)
+    )
+    (property "Value" "+3.3V" (at 160.528 65.024 0)
+      (effects (font (size 1.27 1.27)))
+    )
+    (property "Footprint" "" (at 156.464 64.516 0)
+      (effects (font (size 1.27 1.27)) hide)
+    )
+    (property "Datasheet" "" (at 156.464 64.516 0)
+      (effects (font (size 1.27 1.27)) hide)
+    )
+    (pin "1")
+    (instances
+      (project "BarometerBoard"
+        (path "/0fb9836c-093c-4923-9fd8-054e13e1cd18"
+          (reference "#PWR08") (unit 1)
+        )
+      )
+      (project "Ricardo-Stark"
+        (path "/7db990e4-92e1-4f99-b4d2-435bbec1ba83"
+          (reference "#PWR06") (unit 1)
+        )
+      )
+    )
+  )
   (symbol (lib_id "Connector:TestPoint") (at 188.468 101.854 90) (unit 1)
     (in_bom yes) (on_board yes) (dnp no)
@@
         (path "/7db990e4-92e1-4f99-b4d2-435bbec1ba83"
           (reference "#PWR06") (unit 1)
+        )
+      )
+    )
+  )
+  (symbol (lib_id "Connector:Conn_01x04_Pin") (at 148.59 64.516 0) (unit 1)
+    (in_bom yes) (on_board yes) (dnp no) (fields_autoplaced)
+    (property "Reference" "J2" (at 149.225 56.388 0)
+      (effects (font (size 1.27 1.27)) hide)
+    )
+    (property "Value" "Conn_01x04_Pin" (at 149.225 58.928 0)
+      (effects (font (size 1.27 1.27)) hide)
+    )
+    (property "Footprint" "Connector_JST:JST_SH_SM04B-SRSS-TB_1x04-1MP_P1.00mm_Horizontal" (at 148.59 64.516 0)
+      (effects (font (size 1.27 1.27)) hide)
+    )
+    (property "Datasheet" "~" (at 148.59 64.516 0)
+      (effects (font (size 1.27 1.27)) hide)
+    )
+    (pin "3")
+    (pin "2")
+    (pin "4")
+    (pin "1")
+    (instances
+      (project "BarometerBoard"
+        (path "/0fb9836c-093c-4923-9fd8-054e13e1cd18"
+          (reference "J2") (unit 1)
         )
       )
@@
         )
       )
+    )
+  )
+  (symbol (lib_name "GND_1") (lib_id "power:GND") (at 156.718 61.976 90) (unit 1)
+    (in_bom yes) (on_board yes) (dnp no) (fields_autoplaced)
+    (property "Reference" "#PWR010" (at 163.068 61.976 0)
+      (effects (font (size 1.27 1.27)) hide)
+    )
+    (property "Value" "GND" (at 162.052 61.976 0)
+      (effects (font (size 1.27 1.27)) hide)
+    )
+    (property "Footprint" "" (at 156.718 61.976 0)
+      (effects (font (size 1.27 1.27)) hide)
+    )
+    (property "Datasheet" "" (at 156.718 61.976 0)
+      (effects (font (size 1.27 1.27)) hide)
+    )
+    (pin "1")
+    (instances
+      (project "BarometerBoard"
+        (path "/0fb9836c-093c-4923-9fd8-054e13e1cd18"
+          (reference "#PWR010") (unit 1)
+        )
+      )
